File: ElectronicDesign/ElectronicDesign.kicad_pcb (KiCad board)
At the start: 2 copper layers, 0 parts

Commit message: Update
Parts:
- added C1: 10µ, Capacitor_SMD:C_0805_2012Metric, F.Cu at (96.5, 120.0)
- added C2: 10µ, Capacitor_SMD:C_0805_2012Metric, F.Cu at (100.5, 120.0)
- added C3: 10µ, Capacitor_SMD:C_0805_2012Metric, F.Cu at (84.0, 122.0)
- added C4: 10µ, Capacitor_SMD:C_0805_2012Metric, F.Cu at (79.5, 119.5)
- added C5: 100n, Capacitor_SMD:C_0805_2012Metric, F.Cu at (109.5, 89.0)
- added C6: 100n, Capacitor_SMD:C_0805_2012Metric, F.Cu at (81.2, 90.5)
- added C7: 100n, Capacitor_SMD:C_0805_2012Metric, F.Cu at (81.7, 96.0)
- added C8: 2.2n, Capacitor_SMD:C_0805_2012Metric, F.Cu at (78.2, 93.5)
- added C9: 100n, Capacitor_SMD:C_0805_2012Metric, F.Cu at (130.1, 106.0)
- added ELE10: TestPoint, TestPoint:TestPoint_THTPad_D2.0mm_Drill1.0mm, F.Cu at (92.0, 84.5)
- added ELE11: TestPoint, TestPoint:TestPoint_THTPad_D2.0mm_Drill1.0mm, F.Cu at (96.5, 86.5)
- added ELE3: TestPoint, TestPoint:TestPoint_THTPad_D2.0mm_Drill1.0mm, F.Cu at (109.0, 75.5)
- added ELE4: TestPoint, TestPoint:TestPoint_THTPad_D2.0mm_Drill1.0mm, F.Cu at (106.0, 73.0)
- added ELE5: TestPoint, TestPoint:TestPoint_THTPad_D2.0mm_Drill1.0mm, F.Cu at (102.0, 73.0)
- added ELE6: TestPoint, TestPoint:TestPoint_THTPad_D2.0mm_Drill1.0mm, F.Cu at (97.5, 73.5)
- added ELE7: TestPoint, TestPoint:TestPoint_THTPad_D2.0mm_Drill1.0mm, F.Cu at (94.0, 74.5)
- added ELE8: TestPoint, TestPoint:TestPoint_THTPad_D2.0mm_Drill1.0mm, F.Cu at (91.5, 77.0)
- added ELE9: TestPoint, TestPoint:TestPoint_THTPad_D2.0mm_Drill1.0mm, F.Cu at (91.0, 80.5)
- added R1: 5.1k, Resistor_SMD:R_0805_2012Metric, F.Cu at (100.1, 127.5)
- added R2: 5.1k, Resistor_SMD:R_0805_2012Metric, F.Cu at (123.5, 115.0)
- added R3: 2k, Resistor_SMD:R_0805_2012Metric, F.Cu at (105.1, 125.5)
- added R4: 4.7k, Resistor_SMD:R_0805_2012Metric, F.Cu at (101.1, 89.5)
- added R5: 4.7k, Resistor_SMD:R_0805_2012Metric, F.Cu at (115.5, 94.5)
- added R6: 10k, Resistor_SMD:R_0805_2012Metric, F.Cu at (131.1, 97.5)
- added R7: 330, Resistor_SMD:R_0805_2012Metric, F.Cu at (88.0, 103.5)
- added REF**: MountingHole_2.1mm, MountingHole:MountingHole_2.1mm, F.Cu at (108.0, 129.5)
- added REF**: MountingHole_2.1mm, MountingHole:MountingHole_2.1mm, F.Cu at (120.0, 79.5)
- added REF**: MountingHole_2.1mm, MountingHole:MountingHole_2.1mm, F.Cu at (81.5, 79.5)
- added TP1: 3v3, TestPoint:TestPoint_Pad_D1.5mm, F.Cu at (124.1, 93.6)
- added TP15: ELE0, TestPoint:TestPoint_THTPad_D2.0mm_Drill1.0mm, F.Cu at (112.5, 86.5)
- added TP16: ELE1, TestPoint:TestPoint_THTPad_D2.0mm_Drill1.0mm, F.Cu at (112.5, 82.5)
- added TP17: ELE2, TestPoint:TestPoint_THTPad_D2.0mm_Drill1.0mm, F.Cu at (111.5, 79.0)
- added TP2: TxD0, TestPoint:TestPoint_Pad_D1.5mm, F.Cu at (124.1, 97.1)
- added TP3: RxD0, TestPoint:TestPoint_Pad_D1.5mm, F.Cu at (124.1, 100.1)
- added TP4: IO0, TestPoint:TestPoint_Pad_D1.5mm, F.Cu at (124.1, 103.1)
- added TP5: EN, TestPoint:TestPoint_Pad_D1.5mm, F.Cu at (124.1, 106.1)
- added TP6: GND, TestPoint:TestPoint_Pad_D1.5mm, F.Cu at (124.1, 109.1)
- added U1: ESP32-WROOM-32E, mylib:WIFI-SMD_ESP32-WROOM-32E, F.Cu at (100.5, 108.0)
- added U2: MPR121QR2, mylib:QFN-20_L3.0-W3.0-P0.40-BL, F.Cu at (102.2, 82.9)
- added U3: MPU-6050_C24112, mylib:QFN-24_L4.0-W4.0-P0.50-BL-EP2.7, F.Cu at (81.1, 85.2)
- added U4: TP4056, mylib:ESOP-8_L4.9-W3.9-P1.27-LS6.0-BL-EP, F.Cu at (94.5, 125.5)
- added U5: AMS1117-3.3, mylib:SOT-223-3_L6.5-W3.4-P2.30-LS7.0-BR, F.Cu at (72.5, 100.0)
- added U6: S2B-PH-K-S, mylib:CONN-TH_S2B-PH-K-S-LF-SN, B.Cu at (87.0, 125.3)
- added U7: SS12D10G5, mylib:SW-TH_SHOU-HAN_SS12D10G4, F.Cu at (78.0, 110.3)
- added USBC1: TYPE-C-31-M-12, mylib:USB-C_SMD-TYPE-C-31-M-12_1, F.Cu at (115.0, 122.8)
Routing:
- net GND: track 0.00 -> 235.1 mm, vias 0 -> 6
- net +3V3: track 0.00 -> 136.4 mm, vias 0 -> 2
- net /SDA: track 0.00 -> 74.3 mm, vias 0 -> 4
- net /EN: track 0.00 -> 69.0 mm, vias 0 -> 2
- net /SCL: track 0.00 -> 65.4 mm, vias 0 -> 4
- net Net-(U4-CE): track 0.00 -> 41.1 mm, vias 0 -> 3
- net /INT_GYRO: track 0.00 -> 39.3 mm, vias 0 -> 4
- net /IRQ_TS: track 0.00 -> 35.9 mm, vias 0 -> 2
- net Net-(C3-Pad1): track 0.00 -> 23.8 mm
- net Net-(U4-BAT): track 0.00 -> 23.7 mm, vias 0 -> 2
- net /IO0: track 0.00 -> 22.2 mm
- net Net-(U3-REGOUT): track 0.00 -> 21.1 mm, vias 0 -> 2
- net Net-(U5-VIN): track 0.00 -> 20.5 mm, vias 0 -> 2
- net /TxDO: track 0.00 -> 16.9 mm
- net Net-(USBC1-CC1): track 0.00 -> 16.5 mm
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- added copper zone on B.Cu, net GND
- added copper zone on F.Cu, net GND
Other:
- board outline added: 71.1 x 71.1 mm
- board text added: "LA"
- board text added: "MIDI CONTROLLER"
