File: ElectronicDesign/ElectronicDesign.kicad_sch (KiCad schematic)
At the start: 1 part, among them U1 ESP32-WROOM-32E

Commit message: Update
Parts:
- added C1, C2, C3, C4: 10µ, Capacitor_SMD:C_0805_2012Metric, symbol Device:C
- added C5, C6, C7, C9: 100n, Capacitor_SMD:C_0805_2012Metric, symbol Device:C
- added C8: 2.2n, Capacitor_SMD:C_0805_2012Metric, symbol Device:C
- added D1: LED RED, LED_SMD:LED_0805_2012Metric, symbol Device:LED
- added ELE10, ELE11, ELE3, ELE4, ELE5, ELE6, ELE7, ELE8, ELE9: TestPoint, TestPoint:TestPoint_THTPad_D2.0mm_Drill1.0mm, symbol Connector:TestPoint
- added R1, R2: 5.1k, Resistor_SMD:R_0805_2012Metric, symbol Device:R
- added R3: 2k, Resistor_SMD:R_0805_2012Metric, symbol Device:R
- added R4, R5: 4.7k, Resistor_SMD:R_0805_2012Metric, symbol Device:R
- added R6: 10k, Resistor_SMD:R_0805_2012Metric, symbol Device:R
- added R7: 330, Resistor_SMD:R_0805_2012Metric, symbol Device:R
- added TP1: 3v3, TestPoint:TestPoint_Pad_D1.5mm, symbol Connector:TestPoint
- added TP15: ELE0, TestPoint:TestPoint_THTPad_D2.0mm_Drill1.0mm, symbol Connector:TestPoint
- added TP16: ELE1, TestPoint:TestPoint_THTPad_D2.0mm_Drill1.0mm, symbol Connector:TestPoint
- added TP17: ELE2, TestPoint:TestPoint_THTPad_D2.0mm_Drill1.0mm, symbol Connector:TestPoint
- added TP2: TxD0, TestPoint:TestPoint_Pad_D1.5mm, symbol Connector:TestPoint
- added TP3: RxD0, TestPoint:TestPoint_Pad_D1.5mm, symbol Connector:TestPoint
- added TP4: IO0, TestPoint:TestPoint_Pad_D1.5mm, symbol Connector:TestPoint
- added TP5: EN, TestPoint:TestPoint_Pad_D1.5mm, symbol Connector:TestPoint
- added TP6: GND, TestPoint:TestPoint_Pad_D1.5mm, symbol Connector:TestPoint
- added U2: MPR121QR2, mylib:QFN-20_L3.0-W3.0-P0.40-BL, symbol mylib:MPR121QR2
- added U3: MPU-6050_C24112, mylib:QFN-24_L4.0-W4.0-P0.50-BL-EP2.7, symbol mylib:MPU-6050_C24112
- added U4: TP4056, mylib:ESOP-8_L4.9-W3.9-P1.27-LS6.0-BL-EP, symbol mylib:TP4056
- added U5: AMS1117-3.3, mylib:SOT-223-3_L6.5-W3.4-P2.30-LS7.0-BR, symbol mylib:AMS1117-3.3
- added U6: S2B-PH-K-S, mylib:CONN-TH_S2B-PH-K-S-LF-SN, symbol mylib:S2B-PH-K-S
- added U7: SS12D10G5, mylib:SW-TH_SHOU-HAN_SS12D10G4, symbol mylib:SS12D10G5
- added USBC1: TYPE-C-31-M-12, mylib:USB-C_SMD-TYPE-C-31-M-12_1, symbol mylib:TYPE-C-31-M-12
Connections:
- net GND: now reaches U1.1 (GND)
- net GND: now also U1.15 (GND), U1.38 (GND), U1.39 (GND), C1.2, C2.2, C3.2, C4.1, C5.2, C6.2, C7.2, C8.1, C9.2, D1.1 (K), R1.2, R2.2, R3.2, TP6.1, U2.4 (ADDR), U2.6 (VSS), U2.7 (REXT), U3.1 (CLKIN), U3.11 (FSYNC), U3.18 (GND), U3.25 (EP), U3.9 (AD0), U4.1 (TEMP), U4.3 (GND), U4.9 (EP), U5.1 (GND), USBC1.1 (EH), USBC1.2 (EH), USBC1.3 (EH), USBC1.4 (EH), USBC1.A1B12 (GND), USBC1.B1A12 (GND)
- net at U1.10 (IO25): now also R7.2
- net INT_GYRO: now reaches U1.13 (IO14)
- net INT_GYRO: now also U3.12 (INT)
- net IRQ_TS: now reaches U1.16 (IO13)
- net IRQ_TS: now also U2.1 (~{IRQ})
- net +3V3: now reaches U1.2 (3V3)
- net +3V3: now also C4.2, C6.1, R4.1, R5.1, R6.1, TP1.1, U2.20 (VDD), U3.13 (VDD), U3.8 (VLOGIC), U5.2 (VOUT), U5.4 (VOUT)
- net IO0: now reaches U1.25 (IO0)
- net IO0: now also TP4.1
- net EN: now reaches U1.3 (EN)
- net EN: now also C9.1, R6.2, TP5.1
- net SDA: now reaches U1.33 (IO21)
- net SDA: now also R5.2, U2.3 (SDA), U3.24 (SDA)
- net RXD0: now reaches U1.34 (RXD0)
- net RXD0: now also TP3.1
- net TxDO: now reaches U1.35 (TXD0)
- net TxDO: now also TP2.1
- net SCL: now reaches U1.36 (IO22)
- net SCL: now also R4.2, U2.2 (SCL), U3.23 (SCL)
- new net: U5.3 (VIN), U7.3
- new net: C2.1, U4.5 (BAT), U6.1
- new net: C3.1, U6.2, U7.2
- new net: ELE5.1, U2.13 (ELE5)
- new net: ELE7.1, U2.15 (ELE7)
- new net: ELE4.1, U2.12 (ELE4)
- new net: R2.1, USBC1.B5 (CC2)
- new net: C1.1, U4.4 (VCC), U4.8 (CE), USBC1.A4B9 (VBUS), USBC1.B4A9 (VBUS)
- new net: R1.1, USBC1.A5 (CC1)
- new net: TP16.1, U2.9 (ELE1)
- new net: TP17.1, U2.10 (ELE2)
- new net: R3.1, U4.2 (PROG)
- new net: C7.1, U3.10 (REGOUT)
- new net: ELE10.1, U2.18 (ELE10)
- new net: ELE3.1, U2.11 (ELE3)
- new net: ELE6.1, U2.14 (ELE6)
- new net: ELE8.1, U2.16 (ELE8)
- new net: ELE9.1, U2.17 (ELE9)
- new net: ELE11.1, U2.19 (ELE11)
- new net: C5.1, U2.5 (VREG)
- new net: TP15.1, U2.8 (ELE0)
- new net: D1.2 (A), R7.1
- new net: C8.2, U3.20 (CPOUT)
- no-connect marks 0 -> 48
Other:
- note added: "micro controller programming pogo connection"
